Commit message: fixed mesh path in zed2i urdf

File: zed_wrapper/urdf/zed_macro.urdf.xacro (robot description, xacro)
@@ -1,5 +1,5 @@
 <?xml version="1.0"?>
 <!--
-// Copyright 2025 Stereolabs
+// Copyright 2026 Stereolabs
 //
 // Licensed under the Apache License, Version 2.0 (the "License");
@@ -16,5 +16,5 @@
 -->
 <robot xmlns:xacro="http://wiki.ros.org/xacro">
-  <xacro:property name="M_PI"     value="3.1415926535897931" />
+  <xacro:property name="M_PI" value="3.1415926535897931" />
   <!--
     Parameters:
@@ -94,4 +94,14 @@
       <xacro:property name="mat" value="0.25 0.25 0.25 1.0" />
     </xacro:if>
+    <xacro:if value="${model == 'zedxnano'}">
+      <xacro:property name="baseline" value="0.018" />
+      <xacro:property name="height" value="0.0305" />
+      <xacro:property name="bottom_slope" value="0.0" />
+      <xacro:property name="screw_offset_x" value="0.0" />
+      <xacro:property name="screw_offset_z" value="-0.01525" />
+      <xacro:property name="optical_offset_x" value="-0.01" />
+      <xacro:property name="mono" value="false" />
+      <xacro:property name="mat" value="0.25 0.25 0.25 1.0" />
+    </xacro:if>
     <xacro:if value="${model == 'zedxhdrmini'}">
       <xacro:property name="baseline" value="0.05" />
@@ -130,4 +140,14 @@
       <xacro:property name="screw_offset_x" value="0.0" />
       <xacro:property name="screw_offset_z" value="-0.0155" />
+      <xacro:property name="optical_offset_x" value="-0.005" />
+      <xacro:property name="mono" value="true" />
+      <xacro:property name="mat" value="0.25 0.25 0.25 1.0" />
+    </xacro:if>
+    <xacro:if value="${model == 'zedxones'}">
+      <xacro:property name="baseline" value="0.0" />
+      <xacro:property name="height" value="0.025" />
+      <xacro:property name="bottom_slope" value="0.0" />
+      <xacro:property name="screw_offset_x" value="0.0" />
+      <xacro:property name="screw_offset_z" value="-0.0125" />
       <xacro:property name="optical_offset_x" value="0.0" />
       <xacro:property name="mono" value="true" />
@@ -160,16 +180,16 @@
       <xacro:unless value="${model == 'virtual'}">
         <visual>
-          <origin xyz="${screw_offset_x} 0 ${screw_offset_z}" rpy="0 0 0"/>
+          <origin xyz="${screw_offset_x} 0 ${screw_offset_z}" rpy="0 0 0" />
           <geometry>
-            <mesh filename="file://$(find zed_msgs)/meshes/${model}.stl"/>
+            <mesh filename="package://zed_description/meshes/${model}.stl" />
           </geometry>
-            <material name="zed_mat">
-              <color rgba="${mat}"/>
-            </material>
+          <material name="cam_mat">
+            <color rgba="${mat}" />
+          </material>
         </visual>
         <collision>
-          <origin xyz="${screw_offset_x} 0 ${screw_offset_z}" rpy="0 0 0"/>
+          <origin xyz="${screw_offset_x} 0 ${screw_offset_z}" rpy="0 0 0" />
           <geometry>
-            <mesh filename="file://$(find zed_msgs)/meshes/${model}.stl"/>
+            <mesh filename="package://zed_description/meshes/${model}.stl" />
           </geometry>
         </collision>
@@ -177,6 +197,6 @@
     </link>
     <joint name="${name}_camera_center_joint" type="fixed">
-      <parent link="${name}_camera_link"/>
-      <child link="${name}_camera_center"/>
+      <parent link="${name}_camera_link" />
+      <child link="${name}_camera_center" />
       <origin xyz="0 0 ${height/2}" rpy="0 ${bottom_slope} 0" />
     </joint>
@@ -186,16 +206,16 @@
         <xacro:if value="${model == 'virtual'}">
           <visual>
-            <origin xyz="0 0 0" rpy="0 0 0"/>
+            <origin xyz="0 0 0" rpy="0 0 0" />
             <geometry>
-              <mesh filename="file://$(find zed_msgs)/meshes/${model}.stl"/>
+              <mesh filename="package://zed_description/meshes/${model}.stl" />
             </geometry>
-            <material name="zed_mat">
-              <color rgba="${mat}"/>
+            <material name="cam_mat">
+              <color rgba="${mat}" />
             </material>
           </visual>
           <collision>
-            <origin xyz="0 0 0" rpy="0 0 0"/>
+            <origin xyz="0 0 0" rpy="0 0 0" />
             <geometry>
-              <mesh filename="file://$(find zed_msgs)/meshes/${model}.stl"/>
+              <mesh filename="package://zed_description/meshes/${model}.stl" />
             </geometry>
           </collision>
@@ -203,13 +223,13 @@
       </link>
       <joint name="${name}_left_camera_joint" type="fixed">
-        <parent link="${name}_camera_center"/>
-        <child link="${name}_left_camera_frame"/>
+        <parent link="${name}_camera_center" />
+        <child link="${name}_left_camera_frame" />
         <origin xyz="${optical_offset_x} ${baseline/2} 0" rpy="0 0 0" />
       </joint>
-      <link name="${name}_left_camera_frame_optical"/>
-      <joint name="${name}_left_camera_joint_optical" type="fixed">
-        <origin xyz="0 0 0" rpy="-${M_PI/2} 0.0 -${M_PI/2}"/>
-        <parent link="${name}_left_camera_frame"/>
-        <child link="${name}_left_camera_frame_optical"/>
+      <link name="${name}_left_camera_frame_optical" />
+      <joint name="${name}_left_camera_optical_joint" type="fixed">
+        <origin xyz="0 0 0" rpy="-${M_PI/2} 0.0 -${M_PI/2}" />
+        <parent link="${name}_left_camera_frame" />
+        <child link="${name}_left_camera_frame_optical" />
       </joint>
       <!-- Right Camera -->
@@ -217,16 +237,16 @@
         <xacro:if value="${model == 'virtual'}">
           <visual>
-            <origin xyz="0 0 0" rpy="0 0 0"/>
+            <origin xyz="0 0 0" rpy="0 0 0" />
             <geometry>
-              <mesh filename="file://$(find zed_msgs)/meshes/${model}.stl"/>
+              <mesh filename="package://zed_description/meshes/${model}.stl" />
             </geometry>
-            <material name="zed_mat">
-              <color rgba="${mat}"/>
+            <material name="cam_mat">
+              <color rgba="${mat}" />
             </material>
           </visual>
           <collision>
-            <origin xyz="0 0 0" rpy="0 0 0"/>
+            <origin xyz="0 0 0" rpy="0 0 0" />
             <geometry>
-              <mesh filename="file://$(find zed_msgs)/meshes/${model}.stl"/>
+              <mesh filename="package://zed_description/meshes/${model}.stl" />
             </geometry>
           </collision>
@@ -234,13 +254,13 @@
       </link>
       <joint name="${name}_right_camera_joint" type="fixed">
-        <parent link="${name}_camera_center"/>
-        <child link="${name}_right_camera_frame"/>
+        <parent link="${name}_camera_center" />
+        <child link="${name}_right_camera_frame" />
         <origin xyz="${optical_offset_x} -${baseline/2} 0" rpy="0 0 0" />
       </joint>
-      <link name="${name}_right_camera_frame_optical"/>
-      <joint name="${name}_right_camera_joint_optical" type="fixed">
-        <origin xyz="0 0 0" rpy="-${M_PI/2} 0.0 -${M_PI/2}"/>
-        <parent link="${name}_right_camera_frame"/>
-        <child link="${name}_right_camera_frame_optical"/>
+      <link name="${name}_right_camera_frame_optical" />
+      <joint name="${name}_right_camera_optical_joint" type="fixed">
+        <origin xyz="0 0 0" rpy="-${M_PI/2} 0.0 -${M_PI/2}" />
+        <parent link="${name}_right_camera_frame" />
+        <child link="${name}_right_camera_frame_optical" />
       </joint>
       <!-- ZED2 Sensors -->
@@ -248,24 +268,24 @@
         <link name="${name}_mag_link" />
         <joint name="${name}_mag_joint" type="fixed">
-          <parent link="${name}_camera_center"/>
-          <child link="${name}_mag_link"/>
+          <parent link="${name}_camera_center" />
+          <child link="${name}_mag_link" />
           <origin xyz="0 0 0" rpy="0 0 0" />
         </joint>
         <link name="${name}_baro_link" />
         <joint name="${name}_baro_joint" type="fixed">
-          <parent link="${name}_camera_center"/>
-          <child link="${name}_baro_link"/>
+          <parent link="${name}_camera_center" />
+          <child link="${name}_baro_link" />
           <origin xyz="0 0 0" rpy="0 0 0" />
         </joint>
         <link name="${name}_temp_left_link" />
         <joint name="${name}_temp_left_joint" type="fixed">
-          <parent link="${name}_left_camera_frame"/>
-          <child link="${name}_temp_left_link"/>
+          <parent link="${name}_left_camera_frame" />
+          <child link="${name}_temp_left_link" />
           <origin xyz="0 0 0" rpy="0 0 0" />
         </joint>
         <link name="${name}_temp_right_link" />
         <joint name="${name}_temp_right_joint" type="fixed">
-          <parent link="${name}_right_camera_frame"/>
-          <child link="${name}_temp_right_link"/>
+          <parent link="${name}_right_camera_frame" />
+          <child link="${name}_temp_right_link" />
           <origin xyz="0 0 0" rpy="0 0 0" />
         </joint>
@@ -276,13 +296,13 @@
       <link name="${name}_camera_frame" />
       <joint name="${name}_camera_joint" type="fixed">
-        <parent link="${name}_camera_center"/>
-        <child link="${name}_camera_frame"/>
+        <parent link="${name}_camera_center" />
+        <child link="${name}_camera_frame" />
         <origin xyz="${optical_offset_x} 0 0" rpy="0 0 0" />
       </joint>
-      <link name="${name}_camera_frame_optical"/>
+      <link name="${name}_camera_frame_optical" />
       <joint name="${name}_camera_optical_joint" type="fixed">
-        <origin xyz="0 0 0" rpy="-${M_PI/2} 0.0 -${M_PI/2}"/>
-        <parent link="${name}_camera_frame"/>
-        <child link="${name}_camera_frame_optical"/>
+        <origin xyz="0 0 0" rpy="-${M_PI/2} 0.0 -${M_PI/2}" />
+        <parent link="${name}_camera_frame" />
+        <child link="${name}_camera_frame_optical" />
       </joint>
     </xacro:if>
@@ -290,6 +310,6 @@
       <link name="${name}_gnss_link" />
       <joint name="${name}_gnss_joint" type="fixed">
-        <parent link="${name}_camera_link"/>
-        <child link="${name}_gnss_link"/>
+        <parent link="${name}_camera_link" />
+        <child link="${name}_gnss_link" />
         <xacro:insert_block name="gnss_origin" />
       </joint>
